File: 2Wheel_balance_robot/PCB Layout/Version 2 complete.kicad_pcb (KiCad board)
At the start: 2 copper layers, 56 parts, among them J1 Conn_01x04, J2 CONN_MPU6050, J3 USB_C_Receptacle_USB2.0_14P, J4 ESP_Conn, J5 BATT_CONN, J6 M1_CONN, J7 M2_CONN, J8 ENCODER_CONN, J9 MT6701_CONN, SW2 SW_uP_Reset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

Commit message: done
Parts:
- moved C7 96.0 mm to (134.6, 109.7)
- moved R9 83.2 mm to (140.7, 113.3), turned to 180 degrees
- moved C24 76.4 mm to (111.8, 112.8), turned to -90 degrees
- moved C20 75.1 mm to (110.7, 100.0)
- moved R17 73.9 mm to (142.2, 90.9), turned to 90 degrees
- moved C21 70.8 mm to (102.1, 103.6)
- moved D4 69.5 mm to (144.8, 113.3), turned to 180 degrees
- moved R2 68.9 mm to (132.6, 86.4), turned to 90 degrees
- moved R1 66.6 mm to (100.6, 113.8), turned to 180 degrees
- moved C1 64.5 mm to (93.5, 92.5), turned to 90 degrees
- moved R4 62.7 mm to (105.2, 115.3)
- moved R3 62.6 mm to (105.2, 112.3)
- moved C2 60.6 mm to (90.9, 92.5), turned to 90 degrees
- moved C6 60.2 mm to (99.0, 94.0)
- moved C22 60.0 mm to (115.3, 79.2), turned to 90 degrees
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Routing:
- net +3.3V: track 0.00 -> 73.0 mm
- net /USB_D+: track 0.00 -> 22.7 mm, vias 0 -> 2
- net +5V: track 0.00 -> 18.2 mm
- net /USB_D-: track 0.00 -> 14.6 mm
- net VM: track 0.00 -> 14.5 mm
- net Vusb: track 0.00 -> 11.8 mm
- net Net-(F1-~-Pad1): track 0.00 -> 11.2 mm
- net /CONN_D-: track 0.00 -> 7.67 mm
- net /MD_AO2: track 0.00 -> 7.64 mm
- net /MD_AO1: track 0.00 -> 6.99 mm
- net /MD_BO2: track 0.00 -> 6.64 mm
- net /MD_BO1: track 0.00 -> 6.37 mm
- net Net-(J3-CC2): track 0.00 -> 3.32 mm
- net Net-(J3-CC1): track 0.00 -> 3.32 mm
- net /CONN_D+: track 0.00 -> 3.09 mm
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